File: resources/how-a-matrix-works/schematics/ghosting_example.kicad_sch (KiCad schematic)
At the start: 8 parts

Commit message: fix schematic annotations and order and update images
Parts:
- added Key1, Key3, Key4: ~, Custom:1u_Cherry_MX1A_5Pin_Switch_Kailh_Socket_with_SK6812MINI-E_cutout, symbol Switch:SW_Push
- added Key2: ~, Custom:1u_Cherry_MX1A_5Pin_Switch_Kailh_Socket_with_SK6812MINI-E_cutout, symbol custom:1u_Cherry_MX_Switch_RGB-SK6812MINI-E_cutout
- Key1, Key2, Key3, Key4: value (none) -> ~
Connections:
- net COLUMN0: now also Key1.1, Key2.1
- net COLUMN1: now also Key3.1, Key4.1
- net ROW0: now also Key1.2, Key3.2
- net ROW1: now also Key2.2, Key4.2
Other:
- note added: "LOW 'Key1' key press detected"
- note added: "LOW 'Key3' key press detected"
- note added: "Scanning COLUMN1 and ROW0"
- note removed: "LOW 'Key0' key press detected"
- moved on the sheet: Key1, Key2, Key3, Key4
