File: resources/how-a-matrix-works/schematics/matrix_scanning_example.kicad_sch (KiCad schematic)
At the start: 40 parts

Commit message: fix matrix walk schematic and update images
Other:
- note added: "LOW (inactive)"
- note added: "Scanning Column0 of Row0"
- note added: "Scanning Column0 of Row1"
- note added: "Scanning Column1 of Row0"
- note added: "Scanning Column1 of Row1"
- note removed: "Scanning Column0 and Row0"
- note removed: "Scanning Column0 and Row1"
- note removed: "Scanning Column1 and Row0"
- note removed: "Scanning Column1 and Row1"
Changed lines of the file:
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@@
 		)
 	)
-	(text "Scanning Column1 and Row0"
+	(text "↓"
+		(exclude_from_sim no)
+		(at 171.196 55.626 0)
+		(effects
+			(font
+				(size 5 5)
+				(color 7 255 92 1)
+			)
+		)
+	)
+	(text "←"
+		(exclude_from_sim no)
+		(at 153.162 59.182 0)
+		(effects
+			(font
+				(size 5 5)
+				(color 7 255 92 1)
+			)
+		)
+	)
+	(text "Scanning Column1 of Row0"
 		(exclude_from_sim no)
 		(at 182.626 27.686 0)
@@
 				(size 1.27 1.27)
 				(color 128 77 0 1)
+			)
+		)
+	)
+	(text "→"
+		(exclude_from_sim no)
+		(at 166.116 52.832 0)
+		(effects
+			(font
+				(size 5 5)
+				(color 7 255 92 1)
+			)
+		)
+	)
+	(text "←"
+		(exclude_from_sim no)
+		(at 165.862 59.182 0)
+		(effects
+			(font
+				(size 5 5)
+				(color 7 255 92 1)
 			)
 		)
@@
 		)
 	)
-	(text "HIGH (inactive)"
+	(text "LOW (inactive)"
 		(exclude_from_sim no)
 		(at 167.894 38.862 0)
@@
 		)
 	)
-	(text "Scanning Column0 and Row1"
+	(text "Scanning Column0 of Row1"
 		(exclude_from_sim no)
 		(at 68.834 104.902 0)
@@
 		)
 	)
-	(text "Scanning Column0 and Row0"
+	(text "Scanning Column0 of Row0"
 		(exclude_from_sim no)
 		(at 69.596 27.686 0)
@@
 				(size 1.27 1.27)
 				(color 128 77 0 1)
+			)
+		)
+	)
+	(text "↓"
+		(exclude_from_sim no)
+		(at 157.226 47.244 0)
+		(effects
+			(font
+				(size 5 5)
+				(color 7 255 92 1)
 			)
 		)
@@
 		)
 	)
-	(text "Scanning Column1 and Row1"
+	(text "Scanning Column1 of Row1"
 		(exclude_from_sim no)
 		(at 203.454 104.902 0)
@@
 		)
 	)
-	(text_box "No current flows through 'Key1' (and 'D1') because 'ROW0' and 'COLUMN0' are both HIGH (same voltage potential)."
+	(text_box "Current continues to flow causing 'COLUMN0' to be pulled 'LOW' ('ROW0' and the inactive 'COLUMN0' are still physically connected)."
 		(exclude_from_sim no)
 		(at 173.99 41.91 0)
@@
 		)
 	)
-	(text_box "No current flows through 'Key4' (and 'D4') because 'ROW1' and 'COLUMN1' are both HIGH (same voltage potential."
+	(text_box "No current flows through 'Key4' (and 'D4') because 'ROW1' and 'COLUMN1' are both HIGH (same voltage potential)."
 		(exclude_from_sim no)
 		(at 232.41 72.39 0)
@@
 	(wire
 		(pts
+			(xy 158.75 50.8) (xy 161.29 50.8)
+		)
+		(stroke
+			(width 0)
+			(type default)
+		)
+	)
+	(wire
+		(pts
 			(xy 106.68 160.02) (xy 106.68 161.29)
 		)
@@
 		)
 		(stroke
-			(width 0)
-			(type default)
-		)
-	)
-	(wire
-		(pts
-			(xy 158.75 50.8) (xy 161.29 50.8)
-		)
-		(stroke
